File: hardware/Casco_EEG_Kicad/Adquisicion.kicad_sch (KiCad schematic)
At the start: 55 parts, among them J1 Jack_Touch-Proof, J10 Jack_Touch-Proof, J2 Jack_Touch-Proof, J3 Jack_Touch-Proof, J4 Jack_Touch-Proof, J5 Jack_Touch-Proof, J6 Jack_Touch-Proof, J7 Jack_Touch-Proof, J8 Jack_Touch-Proof, J9 Jack_Touch-Proof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

Commit message: Cambio jumpers
Parts:
- R1, R10, R2, R3, R4, R5, R6, R7, R8, R9: LCSC PN C114662 -> C4190
- U10, U11, U6, U8, U9: LCSC PN (none) -> C150526
Changed lines of the file:
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@@
 			)
 		)
-		(property "LCSC PN" "C114662"
+		(property "LCSC PN" "C4190"
 			(at 44.45 82.55 90)
 			(effects
@@
 			)
 		)
-		(property "LCSC PN" "C114662"
+		(property "LCSC PN" "C4190"
 			(at 44.45 113.03 90)
 			(effects
@@
 			)
 		)
+		(property "LCSC PN" "C150526"
+			(at 76.2 125.73 0)
+			(effects
+				(font
+					(size 1.27 1.27)
+				)
+				(hide yes)
+			)
+		)
 		(pin "5"
 		)
@@
 			)
 		)
+		(property "LCSC PN" "C150526"
+			(at 74.93 34.29 0)
+			(effects
+				(font
+					(size 1.27 1.27)
+				)
+				(hide yes)
+			)
+		)
 		(pin "5"
 		)
@@
 			)
 		)
-		(property "LCSC PN" "C114662"
+		(property "LCSC PN" "C4190"
 			(at 44.45 143.51 90)
 			(effects
@@
 			)
 		)
-		(property "LCSC PN" "C114662"
+		(property "LCSC PN" "C4190"
 			(at 44.45 158.75 90)
 			(effects
@@
 			)
 		)
-		(property "LCSC PN" "C114662"
+		(property "LCSC PN" "C4190"
 			(at 44.45 173.99 90)
 			(effects
@@
 			)
 		)
+		(property "LCSC PN" "C150526"
+			(at 76.2 64.77 0)
+			(effects
+				(font
+					(size 1.27 1.27)
+				)
+				(hide yes)
+			)
+		)
 		(pin "5"
 		)
@@
 			)
 		)
-		(property "LCSC PN" "C114662"
+		(property "LCSC PN" "C4190"
 			(at 44.45 36.83 90)
 			(effects
@@
 			)
 		)
-		(property "LCSC PN" "C114662"
+		(property "LCSC PN" "C4190"
 			(at 44.45 52.07 90)
 			(effects
@@
 			)
 		)
-		(property "LCSC PN" "C114662"
+		(property "LCSC PN" "C4190"
 			(at 44.45 128.27 90)
 			(effects
@@
 			)
 		)
-		(property "LCSC PN" "C114662"
+		(property "LCSC PN" "C4190"
 			(at 44.45 67.31 90)
 			(effects
@@
 			)
 		)
+		(property "LCSC PN" "C150526"
+			(at 76.2 95.25 0)
+			(effects
+				(font
+					(size 1.27 1.27)
+				)
+				(hide yes)
+			)
+		)
 		(pin "5"
 		)
@@
 			)
 		)
+		(property "LCSC PN" "C150526"
+			(at 76.2 156.21 0)
+			(effects
+				(font
+					(size 1.27 1.27)
+				)
+				(hide yes)
+			)
+		)
 		(pin "5"
 		)
@@
 			)
 		)
-		(property "LCSC PN" "C114662"
+		(property "LCSC PN" "C4190"
 			(at 44.45 97.79 90)
 			(effects
