File: hardware/Casco_EEG_Kicad/Alimentacion.kicad_sch (KiCad schematic)
At the start: 44 parts, among them J15 USB4125-GF-A_REVA2, Q1 FS8205A, SW2 PCM12SMTR, U4 TP4056-42-ESOP8, U5 DW01A, U7 AP2112K-3.3TRG1

Commit message: Agrego convertidor DC/DC REM2A-0505S con modelo 3D, símbolo y footprint
Incluyo librería, footprint y modelo 3D del convertidor DC/DC aislado
REM2A-0505S. Actualizo esquemático de alimentación y PCB.

Co-Authored-By: Claude Opus 4.6 <noreply@anthropic.com>
Parts:
- removed PS2: RP-0505S, Huellas:CONV_RP-0505S, symbol RP0505:RP-0505S
- added PS3: REM2A-0505S, Huellas:CONV_REM2A-0505S, symbol REM2A0505:REM2A-0505S
Connections:
- net GNDPWR: now also PS3.10 (-VOUT)
- net GNDPWR_NOAISL: now also PS3.1 (-VIN)
- net V_BUSP: now also PS3.9 (+VOUT)
- net V_BUSP_NOAISL: now also PS3.16 (+VIN)
- new net: PS3.7 (NC), PS3.8 (NC)
- no-connect marks 3 -> 4
