File: hardware/Casco_EEG_Kicad/Casco_EEG_Kicad.kicad_pcb (KiCad board)
At the start: 2 copper layers, 123 x 64.5 mm, 125 parts, among them J1 Jack_Touch-Proof, J10 Jack_Touch-Proof, J11 FTSH-105-XX-X-DV, J12 Conn_01x01_Pin, J15 USB4125-GF-A_REVA2, J2 Jack_Touch-Proof, J3 Jack_Touch-Proof, J4 Jack_Touch-Proof, J5 Jack_Touch-Proof, J6 Jack_Touch-Proof, J7 Jack_Touch-Proof, J8 Jack_Touch-Proof, J9 Jack_Touch-Proof, Q1 FS8205A, SW1 SW_Push, SW2 PCM12SMTR, U1 ADS1299, U10 TPD2E001DRLR, U11 TPD2E001DRLR, U2 HC-05, U3 LPC845M301JBD48E, U4 TP4056-42-ESOP8, U5 DW01A, U6 TPD2E001DRLR, U7 AP2112K-3.3TRG1, U8 TPD2E001DRLR, U9 TPD2E001DRLR

Commit message: Agrego convertidor DC/DC REM2A-0505S con modelo 3D, símbolo y footprint
Incluyo librería, footprint y modelo 3D del convertidor DC/DC aislado
REM2A-0505S. Actualizo esquemático de alimentación y PCB.

Co-Authored-By: Claude Opus 4.6 <noreply@anthropic.com>
Parts:
- removed PS2: RP-0505S, Huellas:CONV_RP-0505S
- added PS3: REM2A-0505S, Huellas:CONV_REM2A-0505S, F.Cu at (103.8, 120.9)
- moved TP_BAT+1 44.7 mm to (58.0, 147.0)
- moved NT2 40.0 mm to (73.0, 103.5)
- moved H4 22.0 mm to (202.5, 103.5)
- moved C30 13.6 mm to (112.0, 104.5)
- moved D3 13.6 mm to (112.0, 99.8)
- moved D4 13.6 mm to (112.0, 98.1)
- moved R21 13.6 mm to (112.0, 102.9)
- moved R22 13.6 mm to (112.0, 101.4)
- moved R23 13.6 mm to (112.0, 96.5)
- moved U4 13.4 mm to (111.3, 109.3)
- moved Q1 13.2 mm to (116.5, 109.5)
- moved R24 11.3 mm to (99.0, 101.5), turned to 90 degrees
- moved U5 11.2 mm to (106.5, 101.0), turned to 180 degrees
- moved R27 10.4 mm to (97.5, 112.5)
- moved R20 10.3 mm to (100.5, 101.5), turned to 90 degrees
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Routing:
- net /Alimentacion/VOUT+: track 153.0 -> 111.0 mm
- net /Alimentacion/V_BUSP: track 49.7 -> 18.3 mm
- net +3.3V: track 170.3 -> 143.0 mm
- net /Alimentacion/V_BUSP_NOAISL: track 12.7 -> 0.00 mm
- net Net-(U7-VOUT): track 17.2 -> 6.37 mm
- net Net-(J15-CC2): track 10.4 -> 0.00 mm
- net Net-(J15-CC1): track 6.63 -> 0.00 mm
- net /Alimentacion/V_BAT_N: track 23.1 -> 19.3 mm
- net Net-(D2-K): track 22.9 -> 20.7 mm
- net GNDPWR: track 16.7 -> 14.9 mm, vias 38 -> 27
- net GNDPWR_NOAISL: vias 7 -> 0
- net GNDD: vias 91 -> 84
- removed copper zone on B.Cu, net GNDPWR
- removed copper zone on F.Cu, net GNDPWR
- removed copper zone on B.Cu, net GNDPWR_NOAISL
- removed copper zone on F.Cu, net GNDPWR_NOAISL
